Commit message: Add moveit (now working)

File: jaco_model/urdf/jaco_arm_old.xacro (robot description, xacro)
@@ -27,6 +27,6 @@
   <property name="api_origin" value="jaco_api_origin" />
   <property name="joint_base" value="jaco_joint_base" />
-  <property name="joint_base_axis_xyz" value="0 0 0.88265" />
-  <property name="joint_base_origin_xyz" value="0 0 0.88265" />
+  <property name="joint_base_axis_xyz" value="0 0 0" />
+  <property name="joint_base_origin_xyz" value="0 0 0" />
   <property name="joint_base_origin_rpy" value="0 0 0" />
   <property name="joint_1" value="jaco_joint_1" />
@@ -95,44 +95,3 @@
     <xacro:jaco_finger_joint joint_name="${joint_finger_3}" type="revolute" parent="${link_hand}" child="${link_finger_3}" joint_axis_xyz="${joint_finger_3_axis_xyz}" joint_origin_xyz="${joint_finger_3_origin_xyz}" joint_origin_rpy="${joint_finger_3_origin_rpy}" lower_limit="${joint_finger_3_lower_limit}" upper_limit="${joint_finger_3_upper_limit}"/>
   </xacro:macro>
-  <joint name="jointarmtoholder" type="fixed">
-    <parent link="${link_base}"/>
-    <child link="holder"/>
-    <origin xyz="0 0 0" rpy="0 0 0" />
-  </joint>
- <link name="holder">
-    <visual>
-      <geometry>
-        <box size="0.04445 0.04445 0.14605"/>
-      </geometry>
-      <origin rpy="0 0 0" xyz="0.0 0 -0.073025"/>
-      <material name="metal">
-        <color rgba="0.5 0.5 0.5 1"/>
-      </material>
-    </visual>
-    <collision>
-      <geometry>
-        <box size="0.53 0.52 0.1"/>
-      </geometry>
-      <origin rpy="0 0 0" xyz="0.0 0 0.1"/>
-    </collision>
-    <inertial>
-      <mass value="150"/>
-      <inertia ixx="0.4" iyy="0.4" izz="0.2" ixy="0.0" ixz="0.0" iyz="0.0"/>
-    </inertial>
-  </link>
-  <link name="table">
-    <visual>
-      <geometry>
-        <box size="1.3716 0.796925 0.7366"/>
-      </geometry>
-      <material name="table_mat">
-        <color rgba="0.5 0.5 0.25 1"/>
-      </material>
-    </visual>
-  </link>
-  <joint name="holder_to_table" type="fixed">
-    <parent link="holder"/>
-    <child link="table"/>
-    <origin xyz="0.663575 0.3762375 -0.51435"/>
-  </joint>
 </root>

File: jaco_model/urdf/standalone_arm.urdf (robot description, URDF)
Before this commit: robot jaco, 11 links, 10 joints
Links:
- added link holder, mass 150; collision box size=0.53 0.52 0.1; visual box size=0.04445 0.04445 0.14605
- added link jaco_api_origin
- added link jaco_end_effector
- added link table; visual box size=1.3716 0.796925 0.7366
Joints:
- added joint holder_to_table: type fixed, parent holder, child table, origin xyz=0.663575 0.3762375 -0.51435
- added joint jaco_link_base_to_api_origin: type fixed, parent jaco_link_base, child jaco_api_origin, origin xyz=0 0 0.028 rpy=0 0 0
- added joint jaco_link_hand_to_end_effector: type fixed, parent jaco_link_hand, child jaco_end_effector, origin xyz=0 0 -0.1687 rpy=0 3.14159265359 0
- added joint jointarmtoholder: type fixed, parent jaco_link_base, child holder, origin xyz=0 0 0 rpy=0 0 0
- joint jaco_joint_1: limit (none) -> lower=-6.28318530718 upper=6.28318530718 effort=30 velocity=0.35
- joint jaco_joint_2: limit (none) -> lower=-3.14159265359 upper=0.0 effort=30 velocity=0.35; type continuous -> revolute
- joint jaco_joint_3: limit (none) -> lower=-3.92699081699 upper=0.785398163397 effort=30 velocity=0.35; type continuous -> revolute
- joint jaco_joint_4: limit (none) -> lower=-6.28318530718 upper=6.28318530718 effort=30 velocity=0.35
- joint jaco_joint_5: limit (none) -> lower=-6.28318530718 upper=6.28318530718 effort=30 velocity=0.35
- joint jaco_joint_6: limit (none) -> lower=-6.28318530718 upper=6.28318530718 effort=30 velocity=0.35
- joint jaco_joint_base: axis 0 0 0 -> 0 0 0.88265; limit (none) -> lower=0 upper=0 effort=30 velocity=0.35; origin xyz=0 0 0 rpy=0 0 0 -> xyz=0 0 0.88265 rpy=0 0 0
