Commit message: add models and positions

File: jaco_model/urdf/jaco_arm_chair.xacro (robot description, xacro)
@@ -28,5 +28,5 @@
   <property name="joint_base" value="jaco_joint_base" />
   <property name="joint_base_axis_xyz" value="0 0 0" />
-  <property name="joint_base_origin_xyz" value="0 0 0" />
+  <property name="joint_base_origin_xyz" value="0.15 0 0.55" />
   <property name="joint_base_origin_rpy" value="0 0 0" />
   <property name="joint_1" value="jaco_joint_1" />
@@ -95,3 +95,174 @@
     <xacro:jaco_finger_joint joint_name="${joint_finger_3}" type="revolute" parent="${link_hand}" child="${link_finger_3}" joint_axis_xyz="${joint_finger_3_axis_xyz}" joint_origin_xyz="${joint_finger_3_origin_xyz}" joint_origin_rpy="${joint_finger_3_origin_rpy}" lower_limit="${joint_finger_3_lower_limit}" upper_limit="${joint_finger_3_upper_limit}"/>
   </xacro:macro>
+  <joint name="jointarmtochair" type="fixed">
+    <parent link="root"/>
+    <child link="base_link"/>
+    <origin xyz="0 0.4 0.5" rpy="0 0 0" />
+  </joint>
+<link name="base_link">
+    <visual>
+      <geometry>
+        <box size="0.53 0.52 0.1"/>
+      </geometry>
+      <origin rpy="0 0 0" xyz="0.0 0 0.1"/>
+      <material name="leather">
+        <color rgba="0.5 0.5 0.5 1"/>
+        <!--texture filename="package://jaco_description/urdf/leather.jpg" /-->
+      </material>
+    </visual>
+    <collision>
+      <geometry>
+        <box size="0.53 0.52 0.1"/>
+      </geometry>
+      <origin rpy="0 0 0" xyz="0.0 0 0.1"/>
+    </collision>
+    <inertial>
+      <mass value="150"/>
+      <inertia ixx="0.4" iyy="0.4" izz="0.2" ixy="0.0" ixz="0.0" iyz="0.0"/>
+    </inertial>
+  </link>
+  <link name="back">
+    <visual>
+      <geometry>
+        <box size="0.1 0.43 0.52"/>
+      </geometry>
+      <!--origin rpy="0 0 0" xyz="-0.5 0 0.3"/-->
+      <material name="leather"/>
+    </visual>
+  </link>
+  <joint name="base_link_to_back" type="fixed">
+    <parent link="base_link"/>
+    <child link="back"/>
+    <origin xyz="-0.28 0 0.375"/>
+  </joint>
+   <link name="back_head">
+    <visual>
+      <geometry>
+        <box size="0.1 0.23 0.18"/>
+      </geometry>
+      <!--origin rpy="0 0 0" xyz="-0.5 0 0.3"/-->
+      <material name="leather"/>
+    </visual>
+  </link>
+  <joint name="base_link_to_back_head" type="fixed">
+    <parent link="base_link"/>
+    <child link="back_head"/>
+    <origin xyz="-0.28 0 0.7"/>
+  </joint>
+ <!--arm rests-->
+  <link name="arm_rest_right">
+    <visual>
+      <geometry>
+        <box size="0.41 0.07 0.05"/>
+      </geometry>
+      <!--origin rpy="0 0 0" xyz="-0.5 0 0.3"/-->
+      <material name="leather"/>
+    </visual>
+  </link>
+  <joint name="base_link_to_arm_rest_right" type="fixed">
+    <parent link="base_link"/>
+    <child link="arm_rest_right"/>
+    <origin xyz="-0.06 0.24 0.25"/>
+  </joint>
+ <link name="arm_rest_left">
+    <visual>
+      <geometry>
+        <box size="0.41 0.07 0.05"/>
+      </geometry>
+      <!--origin rpy="0 0 0" xyz="-0.5 0 0.3"/-->
+      <material name="leather"/>
+    </visual>
+  </link>
+  <joint name="base_link_to_arm_rest_left" type="fixed">
+    <parent link="base_link"/>
+    <child link="arm_rest_left"/>
+    <origin xyz="-0.06 -0.24 0.25"/>
+  </joint>
+  <!-- main driving wheels -->
+  <link name="left_wheel">
+    <visual>
+      <geometry>
+        <cylinder length="0.09" radius="0.125"/>
+      </geometry>
+      <origin rpy="1.57075 0 0" xyz="0.0 0.0 0.0"/>
+      <material name="wheel">
+        <color rgba="0.0 0.0 0.9 1"/>
+      </material>
+    </visual>
+    <collision>
+      <geometry>
+        <cylinder length="0.06" radius="0.12"/>
+      </geometry>
+      <origin rpy="1.57075 0 0" xyz="0.0 0.0 0.0"/>
+    </collision>
+  </link>
+  <joint name="base_link_to_left_wheel" type="continuous">
+    <parent link="base_link"/>
+    <child link="left_wheel"/>
+    <origin xyz="0.05 0.3 -0.3"/>
+    <axis xyz="0 1 0"/>
+  </joint>
+  <link name="right_wheel">
+    <visual>
+      <geometry>
+        <cylinder length="0.09" radius="0.125"/>
+      </geometry>
+      <origin rpy="1.57075 0 0" xyz="0.0 0.0 0.0"/>
+      <material name="wheel"/>
+    </visual>
+    <collision>
+      <geometry>
+        <cylinder length="0.06" radius="0.12"/>
+      </geometry>
+      <origin rpy="1.57075 0 0" xyz="0.0 0.0 0.0"/>
+    </collision>
+  </link>
+  <joint name="base_link_to_right_wheel" type="continuous">
+    <parent link="base_link"/>
+    <child link="right_wheel"/>
+    <origin xyz="0.05 -0.3 -0.3"/>
+    <axis xyz="0 1 0"/>
+  </joint>
+ <link name="motor_cage">
+    <visual>
+      <geometry>
+        <box size="0.48 0.34 0.25"/>
+      </geometry>
+      <!--origin rpy="0 0 0" xyz="-0.5 0 0.3"/-->
+      <material name="leather"/>
+    </visual>
+  </link>
+  <joint name="base_link_to_motor_cage" type="fixed">
+    <parent link="base_link"/>
+    <child link="motor_cage"/>
+    <origin xyz="0 0 -0.2"/>
+  </joint>
+ <link name="under_seat">
+    <visual>
+      <geometry>
+        <box size="0.38 0.32 0.04"/>
+      </geometry>
+      <!--origin rpy="0 0 0" xyz="-0.5 0 0.3"/-->
+      <material name="leather"/>
+    </visual>
+  </link>
+  <joint name="base_link_to_under_seat" type="fixed">
+    <parent link="base_link"/>
+    <child link="under_seat"/>
+    <origin xyz="0 0 0"/>
+  </joint>
+  <link name="foot_plate">
+    <visual>
+      <geometry>
+        <box size="0.44 0.38 0.05"/>
+      </geometry>
+      <!--origin rpy="0 0 0" xyz="-0.5 0 0.3"/-->
+      <material name="leather"/>
+    </visual>
+  </link>
+  <joint name="base_link_to_foot_plate" type="fixed">
+    <parent link="base_link"/>
+    <child link="foot_plate"/>
+    <origin xyz="0.47 0 -0.3"/>
+  </joint>
 </root>

File: jaco_model/urdf/jaco_arm_table.xacro (robot description, xacro)
@@ -27,6 +27,6 @@
   <property name="api_origin" value="jaco_api_origin" />
   <property name="joint_base" value="jaco_joint_base" />
-  <property name="joint_base_axis_xyz" value="0 0 0" />
-  <property name="joint_base_origin_xyz" value="0 0 0" />
+  <property name="joint_base_axis_xyz" value="0 0 0.88265" />
+  <property name="joint_base_origin_xyz" value="0 0 0.88265" />
   <property name="joint_base_origin_rpy" value="0 0 0" />
   <property name="joint_1" value="jaco_joint_1" />
@@ -95,3 +95,44 @@
     <xacro:jaco_finger_joint joint_name="${joint_finger_3}" type="revolute" parent="${link_hand}" child="${link_finger_3}" joint_axis_xyz="${joint_finger_3_axis_xyz}" joint_origin_xyz="${joint_finger_3_origin_xyz}" joint_origin_rpy="${joint_finger_3_origin_rpy}" lower_limit="${joint_finger_3_lower_limit}" upper_limit="${joint_finger_3_upper_limit}"/>
   </xacro:macro>
+  <joint name="jointarmtoholder" type="fixed">
+    <parent link="${link_base}"/>
+    <child link="holder"/>
+    <origin xyz="0 0 0" rpy="0 0 0" />
+  </joint>
+ <link name="holder">
+    <visual>
+      <geometry>
+        <box size="0.04445 0.04445 0.14605"/>
+      </geometry>
+      <origin rpy="0 0 0" xyz="0.0 0 -0.073025"/>
+      <material name="metal">
+        <color rgba="0.5 0.5 0.5 1"/>
+      </material>
+    </visual>
+    <collision>
+      <geometry>
+        <box size="0.53 0.52 0.1"/>
+      </geometry>
+      <origin rpy="0 0 0" xyz="0.0 0 0.1"/>
+    </collision>
+    <inertial>
+      <mass value="150"/>
+      <inertia ixx="0.4" iyy="0.4" izz="0.2" ixy="0.0" ixz="0.0" iyz="0.0"/>
+    </inertial>
+  </link>
+  <link name="table">
+    <visual>
+      <geometry>
+        <box size="1.3716 0.796925 0.7366"/>
+      </geometry>
+      <material name="table_mat">
+        <color rgba="0.5 0.5 0.25 1"/>
+      </material>
+    </visual>
+  </link>
+  <joint name="holder_to_table" type="fixed">
+    <parent link="holder"/>
+    <child link="table"/>
+    <origin xyz="0.663575 0.3762375 -0.51435"/>
+  </joint>
 </root>

File: jaco_model/urdf/jaco_arm_table2.xacro (robot description, xacro)
@@ -27,6 +27,6 @@
   <property name="api_origin" value="jaco_api_origin" />
   <property name="joint_base" value="jaco_joint_base" />
-  <property name="joint_base_axis_xyz" value="0 0 0" />
-  <property name="joint_base_origin_xyz" value="0 0 0" />
+  <property name="joint_base_axis_xyz" value="0 0 0.88265" />
+  <property name="joint_base_origin_xyz" value="0 0 0.88265" />
   <property name="joint_base_origin_rpy" value="0 0 0" />
   <property name="joint_1" value="jaco_joint_1" />
@@ -95,3 +95,59 @@
     <xacro:jaco_finger_joint joint_name="${joint_finger_3}" type="revolute" parent="${link_hand}" child="${link_finger_3}" joint_axis_xyz="${joint_finger_3_axis_xyz}" joint_origin_xyz="${joint_finger_3_origin_xyz}" joint_origin_rpy="${joint_finger_3_origin_rpy}" lower_limit="${joint_finger_3_lower_limit}" upper_limit="${joint_finger_3_upper_limit}"/>
   </xacro:macro>
+  <joint name="jointarmtoholder" type="fixed">
+    <parent link="${link_base}"/>
+    <child link="holder"/>
+    <origin xyz="0 0 0" rpy="0 0 0" />
+  </joint>
+ <link name="holder">
+    <visual>
+      <geometry>
+        <box size="0.04445 0.04445 0.14605"/>
+      </geometry>
+      <origin rpy="0 0 0" xyz="0.0 0 -0.073025"/>
+      <material name="metal">
+        <color rgba="0.5 0.5 0.5 1"/>
+      </material>
+    </visual>
+    <collision>
+      <geometry>
+        <box size="0.53 0.52 0.1"/>
+      </geometry>
+      <origin rpy="0 0 0" xyz="0.0 0 0.1"/>
+    </collision>
+    <inertial>
+      <mass value="150"/>
+      <inertia ixx="0.4" iyy="0.4" izz="0.2" ixy="0.0" ixz="0.0" iyz="0.0"/>
+    </inertial>
+  </link>
+  <link name="table">
+    <visual>
+      <geometry>
+        <box size="1.3716 0.796925 0.7366"/>
+      </geometry>
+      <material name="table_mat">
+        <color rgba="0.5 0.5 0.25 1"/>
+      </material>
+    </visual>
+  </link>
+  <joint name="holder_to_table" type="fixed">
+    <parent link="holder"/>
+    <child link="table"/>
+    <origin xyz="0.663575 0.3762375 -0.51435"/>
+  </joint>
+  <link name="obstacle">
+    <visual>
+      <geometry>
+        <cylinder length="0.2" radius="0.05"/>
+      </geometry>
+      <material name="obstacle_mat">
+        <color rgba="0.5 0.25 0.5 1"/>
+      </material>
+    </visual>
+  </link>
+  <joint name="table_to_obstacle" type="fixed">
+    <parent link="table"/>
+    <child link="obstacle"/>
+    <origin xyz="-0.35 -0.1 0.5"/>
+  </joint>
 </root>

File: jaco_model/urdf/standalone_arm.urdf (robot description, URDF)
Before this commit: robot jaco, 15 links, 14 joints
Links:
- added link obstacle; visual cylinder length=0.2 radius=0.05
Joints:
- added joint table_to_obstacle: type fixed, parent table, child obstacle, origin xyz=-0.35 -0.1 0.5

File: jaco_model/urdf/standalone_arm.xacro (robot description, xacro)
@@ -13,5 +13,5 @@
     xmlns:physics="http://playerstage.sourceforge.net/gazebo/xmlschema/#physics"
 	xmlns:xacro="http://ros.org/wiki/xacro" name="jaco">
-  <xacro:include filename="$(find jaco_model)/urdf/jaco_arm.xacro" />
+  <xacro:include filename="$(find jaco_model)/urdf/jaco_arm_table2.xacro" />
 <link name="root">
       <visual>

Commit message: IMprove existing models

File: jaco_model/urdf/jaco_arm_chair.xacro (robot description, xacro)
@@ -107,5 +107,5 @@
       <origin rpy="0 0 0" xyz="0.0 0 0.1"/>
       <material name="leather">
-        <color rgba="0.5 0.5 0.5 1"/>
+        <color rgba="0.25 0.5 0.25 1"/>
         <!--texture filename="package://jaco_description/urdf/leather.jpg" /-->
       </material>

File: jaco_model/urdf/jaco_arm_table2.xacro (robot description, xacro)
@@ -149,5 +149,5 @@
     <parent link="table"/>
     <child link="obstacle"/>
-    <origin xyz="-0.35 -0.1 0.5"/>
+    <origin xyz="-0.35 0 0.5"/>
   </joint>
 </root>

File: jaco_model/urdf/standalone_arm.urdf (robot description, URDF)
Before this commit: robot jaco, 16 links, 15 joints
Links:
- removed link holder
- removed link obstacle
- removed link table
- added link arm_rest_left; visual box size=0.41 0.07 0.05
- added link arm_rest_right; visual box size=0.41 0.07 0.05
- added link back; visual box size=0.1 0.43 0.52
- added link back_head; visual box size=0.1 0.23 0.18
- added link base_link, mass 150; collision box size=0.53 0.52 0.1; visual box size=0.53 0.52 0.1
- added link foot_plate; visual box size=0.44 0.38 0.05
- added link left_wheel; collision cylinder length=0.06 radius=0.12; visual cylinder length=0.09 radius=0.125
- added link motor_cage; visual box size=0.48 0.34 0.25
- added link right_wheel; collision cylinder length=0.06 radius=0.12; visual cylinder length=0.09 radius=0.125
- added link under_seat; visual box size=0.38 0.32 0.04
Joints:
- removed joint holder_to_table
- removed joint jointarmtoholder
- removed joint table_to_obstacle
- added joint base_link_to_arm_rest_left: type fixed, parent base_link, child arm_rest_left, origin xyz=-0.06 -0.24 0.25
- added joint base_link_to_arm_rest_right: type fixed, parent base_link, child arm_rest_right, origin xyz=-0.06 0.24 0.25
- added joint base_link_to_back: type fixed, parent base_link, child back, origin xyz=-0.28 0 0.375
- added joint base_link_to_back_head: type fixed, parent base_link, child back_head, origin xyz=-0.28 0 0.7
- added joint base_link_to_foot_plate: type fixed, parent base_link, child foot_plate, origin xyz=0.47 0 -0.3
- added joint base_link_to_left_wheel: type continuous, parent base_link, child left_wheel, origin xyz=0.05 0.3 -0.3, axis 0 1 0
- added joint base_link_to_motor_cage: type fixed, parent base_link, child motor_cage, origin xyz=0 0 -0.2
- added joint base_link_to_right_wheel: type continuous, parent base_link, child right_wheel, origin xyz=0.05 -0.3 -0.3, axis 0 1 0
- added joint base_link_to_under_seat: type fixed, parent base_link, child under_seat, origin xyz=0 0 0
- added joint jointarmtochair: type fixed, parent root, child base_link, origin xyz=0 0.4 0.5 rpy=0 0 0
- joint jaco_joint_base: axis 0 0 0.88265 -> 0 0 0; origin xyz=0 0 0.88265 rpy=0 0 0 -> xyz=0.15 0 0.55 rpy=0 0 0

File: jaco_model/urdf/standalone_arm.xacro (robot description, xacro)
@@ -13,5 +13,5 @@
     xmlns:physics="http://playerstage.sourceforge.net/gazebo/xmlschema/#physics"
 	xmlns:xacro="http://ros.org/wiki/xacro" name="jaco">
-  <xacro:include filename="$(find jaco_model)/urdf/jaco_arm_table2.xacro" />
+  <xacro:include filename="$(find jaco_model)/urdf/jaco_arm_chair.xacro" />
 <link name="root">
       <visual>

Commit message: Fix moveit issues, add hand demos

File: jaco_model/urdf/jaco_arm_chair.xacro (robot description, xacro)
@@ -28,5 +28,5 @@
   <property name="joint_base" value="jaco_joint_base" />
   <property name="joint_base_axis_xyz" value="0 0 0" />
-  <property name="joint_base_origin_xyz" value="0.15 0 0.55" />
+  <property name="joint_base_origin_xyz" value="0 0 0.55" />
   <property name="joint_base_origin_rpy" value="0 0 0" />
   <property name="joint_1" value="jaco_joint_1" />
@@ -98,5 +98,5 @@
     <parent link="root"/>
     <child link="base_link"/>
-    <origin xyz="0 0.4 0.5" rpy="0 0 0" />
+    <origin xyz="0.4 0 0.5" rpy="0 0 ${-1*J_PI/2}" />
   </joint>
 <link name="base_link">

File: jaco_model/urdf/standalone_arm.urdf (robot description, URDF)
Before this commit: robot jaco, 23 links, 22 joints
Joints:
- joint jaco_joint_base: origin xyz=0.15 0 0.55 rpy=0 0 0 -> xyz=0 0 0.55 rpy=0 0 0
- joint jointarmtochair: origin xyz=0 0.4 0.5 rpy=0 0 0 -> xyz=0.4 0 0.5 rpy=0 0 -1.57079632679

Commit message: Fix model, add moveit integration

File: jaco_model/urdf/jaco_arm_chair.xacro (robot description, xacro)
@@ -96,12 +96,12 @@
   </xacro:macro>
   <joint name="jointarmtochair" type="fixed">
-    <parent link="root"/>
+    <parent link="jaco_link_base"/>
     <child link="base_link"/>
-    <origin xyz="0.4 0 0.5" rpy="0 0 ${-1*J_PI/2}" />
+    <origin xyz="0.3 0.1778 0" rpy="0 0 ${-1*J_PI/2}" />
   </joint>
 <link name="base_link">
     <visual>
       <geometry>
-        <box size="0.53 0.52 0.1"/>
+        <box size="0.52 0.51 0.1"/>
       </geometry>
       <origin rpy="0 0 0" xyz="0.0 0 0.1"/>
@@ -163,5 +163,5 @@
     <parent link="base_link"/>
     <child link="arm_rest_right"/>
-    <origin xyz="-0.06 0.24 0.25"/>
+    <origin xyz="-0.12 0.24 0.25"/>
   </joint>
  <link name="arm_rest_left">
@@ -177,5 +177,5 @@
     <parent link="base_link"/>
     <child link="arm_rest_left"/>
-    <origin xyz="-0.06 -0.24 0.25"/>
+    <origin xyz="-0.12 -0.24 0.25"/>
   </joint>
   <!-- main driving wheels -->

File: jaco_model/urdf/standalone_arm.urdf (robot description, URDF)
Before this commit: robot jaco, 23 links, 22 joints
Links:
- link base_link: geometry collision box size=0.53 0.52 0.1; visual box size=0.52 0.51 0.1
Joints:
- joint base_link_to_arm_rest_left: origin xyz=-0.06 -0.24 0.25 -> xyz=-0.12 -0.24 0.25
- joint base_link_to_arm_rest_right: origin xyz=-0.06 0.24 0.25 -> xyz=-0.12 0.24 0.25
- joint jointarmtochair: origin xyz=0.4 0 0.5 rpy=0 0 -1.57079632679 -> xyz=0.3 0.1778 0 rpy=0 0 -1.57079632679; parent root -> jaco_link_base

Commit message: fix issues, add useless files, feel sad

File: jaco_model/urdf/jaco_arm_chair.xacro (robot description, xacro)
@@ -28,5 +28,5 @@
   <property name="joint_base" value="jaco_joint_base" />
   <property name="joint_base_axis_xyz" value="0 0 0" />
-  <property name="joint_base_origin_xyz" value="0 0 0.55" />
+  <property name="joint_base_origin_xyz" value="0 0 0.4826" />
   <property name="joint_base_origin_rpy" value="0 0 0" />
   <property name="joint_1" value="jaco_joint_1" />
@@ -107,6 +107,5 @@
       <origin rpy="0 0 0" xyz="0.0 0 0.1"/>
       <material name="leather">
-        <color rgba="0.25 0.5 0.25 1"/>
-        <!--texture filename="package://jaco_description/urdf/leather.jpg" /-->
+        <color rgba="0.466667 0.533333 0.6 1"/>
       </material>
     </visual>
@@ -197,5 +196,5 @@
     </collision>
   </link>
-  <joint name="base_link_to_left_wheel" type="continuous">
+  <joint name="base_link_to_left_wheel" type="fixed">
     <parent link="base_link"/>
     <child link="left_wheel"/>
@@ -218,5 +217,5 @@
     </collision>
   </link>
-  <joint name="base_link_to_right_wheel" type="continuous">
+  <joint name="base_link_to_right_wheel" type="fixed">
     <parent link="base_link"/>
     <child link="right_wheel"/>
@@ -266,3 +265,19 @@
     <origin xyz="0.47 0 -0.3"/>
   </joint>
+  <link name="table_top">
+    <visual>
+      <geometry>
+        <box size="1.8288 0.6096 0.03175"/>
+      </geometry>
+      <!--origin rpy="0 0 0" xyz="-0.5 0 0.3"/-->
+      <material name="wood">
+        <color rgba="0.627451 0.321569 0.176471 1"/>
+      </material>
+    </visual>
+  </link>
+  <joint name="table_to_arm" type="fixed">
+    <parent link="jaco_link_base"/>
+    <child link="table_top"/>
+    <origin rpy="0 0 0" xyz="0.2794 -0.4826 0.2667"/>
+  </joint>
 </root>

File: jaco_model/urdf/standalone_arm.urdf (robot description, URDF)
Before this commit: robot jaco, 23 links, 22 joints
Links:
- added link table_top; visual box size=1.8288 0.6096 0.03175
Joints:
- added joint table_to_arm: type fixed, parent jaco_link_base, child table_top, origin xyz=0.2794 -0.4826 0.2667 rpy=0 0 0
- joint base_link_to_left_wheel: type continuous -> fixed
- joint base_link_to_right_wheel: type continuous -> fixed
- joint jaco_joint_base: origin xyz=0 0 0.55 rpy=0 0 0 -> xyz=0 0 0.4826 rpy=0 0 0

Commit message: Add camera integration in moveit

File: jaco_model/urdf/jaco_arm_chair.xacro (robot description, xacro)
@@ -28,5 +28,5 @@
   <property name="joint_base" value="jaco_joint_base" />
   <property name="joint_base_axis_xyz" value="0 0 0" />
-  <property name="joint_base_origin_xyz" value="0 0 0.4826" />
+  <property name="joint_base_origin_xyz" value="0 0 0" />
   <property name="joint_base_origin_rpy" value="0 0 0" />
   <property name="joint_1" value="jaco_joint_1" />

File: jaco_model/urdf/jaco_arm_table.xacro (robot description, xacro)
@@ -27,6 +27,6 @@
   <property name="api_origin" value="jaco_api_origin" />
   <property name="joint_base" value="jaco_joint_base" />
-  <property name="joint_base_axis_xyz" value="0 0 0.88265" />
-  <property name="joint_base_origin_xyz" value="0 0 0.88265" />
+  <property name="joint_base_axis_xyz" value="0 0 0" />
+  <property name="joint_base_origin_xyz" value="0 0 0" />
   <property name="joint_base_origin_rpy" value="0 0 0" />
   <property name="joint_1" value="jaco_joint_1" />

File: jaco_model/urdf/standalone_arm.urdf (robot description, URDF)
Before this commit: robot jaco, 24 links, 23 joints
Joints:
- joint jaco_joint_base: origin xyz=0 0 0.4826 rpy=0 0 0 -> xyz=0 0 0 rpy=0 0 0
