Commit message: Add camera integration

File: jaco_model/urdf/jaco_arm_chair_ORIGINAL.xacro (robot description, xacro)
@@ -97,8 +97,8 @@
   <joint name="jointarmtochair" type="fixed">
     <parent link="jaco_link_base"/>
-    <child link="base_link_urdf"/>
+    <child link="base_link"/>
     <origin xyz="0.3 0.1778 0" rpy="0 0 ${-1*J_PI/2}" />
   </joint>
-<link name="base_link_urdf">
+<link name="base_link">
     <visual>
       <geometry>
@@ -130,6 +130,6 @@
     </visual>
   </link>
-  <joint name="base_link_urdf_to_back" type="fixed">
-    <parent link="base_link_urdf"/>
+  <joint name="base_link_to_back" type="fixed">
+    <parent link="base_link"/>
     <child link="back"/>
     <origin xyz="-0.28 0 0.375"/>
@@ -144,6 +144,6 @@
     </visual>
   </link>
-  <joint name="base_link_urdf_to_back_head" type="fixed">
-    <parent link="base_link_urdf"/>
+  <joint name="base_link_to_back_head" type="fixed">
+    <parent link="base_link"/>
     <child link="back_head"/>
     <origin xyz="-0.28 0 0.7"/>
@@ -159,6 +159,6 @@
     </visual>
   </link>
-  <joint name="base_link_urdf_to_arm_rest_right" type="fixed">
-    <parent link="base_link_urdf"/>
+  <joint name="base_link_to_arm_rest_right" type="fixed">
+    <parent link="base_link"/>
     <child link="arm_rest_right"/>
     <origin xyz="-0.12 0.24 0.25"/>
@@ -173,6 +173,6 @@
     </visual>
   </link>
-  <joint name="base_link_urdf_to_arm_rest_left" type="fixed">
-    <parent link="base_link_urdf"/>
+  <joint name="base_link_to_arm_rest_left" type="fixed">
+    <parent link="base_link"/>
     <child link="arm_rest_left"/>
     <origin xyz="-0.12 -0.27 0.25"/>
@@ -196,6 +196,6 @@
     </collision>
   </link>
-  <joint name="base_link_urdf_to_left_wheel" type="fixed">
-    <parent link="base_link_urdf"/>
+  <joint name="base_link_to_left_wheel" type="fixed">
+    <parent link="base_link"/>
     <child link="left_wheel"/>
     <origin xyz="0.05 0.3 -0.3"/>
@@ -217,6 +217,6 @@
     </collision>
   </link>
-  <joint name="base_link_urdf_to_right_wheel" type="fixed">
-    <parent link="base_link_urdf"/>
+  <joint name="base_link_to_right_wheel" type="fixed">
+    <parent link="base_link"/>
     <child link="right_wheel"/>
     <origin xyz="0.05 -0.3 -0.3"/>
@@ -232,6 +232,6 @@
     </visual>
   </link>
-  <joint name="base_link_urdf_to_motor_cage" type="fixed">
-    <parent link="base_link_urdf"/>
+  <joint name="base_link_to_motor_cage" type="fixed">
+    <parent link="base_link"/>
     <child link="motor_cage"/>
     <origin xyz="0 0 -0.2"/>
@@ -246,6 +246,6 @@
     </visual>
   </link>
-  <joint name="base_link_urdf_to_under_seat" type="fixed">
-    <parent link="base_link_urdf"/>
+  <joint name="base_link_to_under_seat" type="fixed">
+    <parent link="base_link"/>
     <child link="under_seat"/>
     <origin xyz="0 0 0"/>
@@ -260,6 +260,6 @@
     </visual>
   </link>
-  <joint name="base_link_urdf_to_foot_plate" type="fixed">
-    <parent link="base_link_urdf"/>
+  <joint name="base_link_to_foot_plate" type="fixed">
+    <parent link="base_link"/>
     <child link="foot_plate"/>
     <origin xyz="0.47 0 -0.3"/>
@@ -298,5 +298,5 @@
     <visual>
       <geometry>
-        <box size="0.27 0.4 0.75"/>
+        <box size="0.19 0.4 0.65"/>
       </geometry>
       <material name="wood">
@@ -305,8 +305,8 @@
     </visual>
   </link>
-  <joint name="base_link_urdf_to_human" type="fixed">
-    <parent link="base_link_urdf"/>
+  <joint name="base_link_to_human" type="fixed">
+    <parent link="base_link"/>
     <child link="human"/>
-    <origin rpy="0 0 0" xyz="-0.08 0.0 0.57"/>
+    <origin rpy="0 0 0" xyz="-0.12 0.0 0.52"/>
   </joint>
 </root>

File: jaco_model/urdf/standalone_arm.urdf (robot description, URDF)
Before this commit: robot jaco, 24 links, 23 joints
Links:
- removed link base_link
- added link base_link_urdf, mass 150; collision box size=0.53 0.52 0.1; visual box size=0.52 0.51 0.1
- added link human; visual box size=0.19 0.4 0.65
- added link right_wall; visual box size=0.1 3.0 3.0
Joints:
- removed joint base_link_to_arm_rest_left
- removed joint base_link_to_arm_rest_right
- removed joint base_link_to_back
- removed joint base_link_to_back_head
- removed joint base_link_to_foot_plate
- removed joint base_link_to_left_wheel
- removed joint base_link_to_motor_cage
- removed joint base_link_to_right_wheel
- removed joint base_link_to_under_seat
- added joint base_link_urdf_to_arm_rest_left: type fixed, parent base_link_urdf, child arm_rest_left, origin xyz=-0.12 -0.27 0.25
- added joint base_link_urdf_to_arm_rest_right: type fixed, parent base_link_urdf, child arm_rest_right, origin xyz=-0.12 0.24 0.25
- added joint base_link_urdf_to_back: type fixed, parent base_link_urdf, child back, origin xyz=-0.28 0 0.375
- added joint base_link_urdf_to_back_head: type fixed, parent base_link_urdf, child back_head, origin xyz=-0.28 0 0.7
- added joint base_link_urdf_to_foot_plate: type fixed, parent base_link_urdf, child foot_plate, origin xyz=0.47 0 -0.3
- added joint base_link_urdf_to_human: type fixed, parent base_link_urdf, child human, origin xyz=-0.12 0.0 0.52 rpy=0 0 0
- added joint base_link_urdf_to_left_wheel: type fixed, parent base_link_urdf, child left_wheel, origin xyz=0.05 0.3 -0.3, axis 0 1 0
- added joint base_link_urdf_to_motor_cage: type fixed, parent base_link_urdf, child motor_cage, origin xyz=0 0 -0.2
- added joint base_link_urdf_to_right_wheel: type fixed, parent base_link_urdf, child right_wheel, origin xyz=0.05 -0.3 -0.3, axis 0 1 0
- added joint base_link_urdf_to_under_seat: type fixed, parent base_link_urdf, child under_seat, origin xyz=0 0 0
- added joint right_wall_to_arm: type fixed, parent jaco_link_base, child right_wall, origin xyz=-0.6 0.0 0.0 rpy=0 0 0
- joint jointarmtochair: child base_link -> base_link_urdf
